File: hw/kicad/base/12V/12V.kicad_pcb (KiCad board)
At the start: 2 copper layers, 45 x 45 mm, 32 parts, among them J1 USB_B_Micro, J2 TOP, J3 XT30PW-M, J4 BUTTOM, U1 LM1117MP-3.3, U2 LM2596S-5, U3 CP2102N-Axx-xQFN28

Commit message: 更换接口线序
Connections:
- net /PWM_5 renamed /GPIO_1
- net /PWM_6 renamed /GPIO_2
- net /PWM_7 renamed /GPIO_3
- net /PWM_8 renamed /GPIO_4
- J2 pad 15: /PWM_1 -> /CAN_H
- J2 pad 16: /PWM_2 -> /CAN_L
- J2 pad 17: /PWM_3 -> /USB+
- J2 pad 18: /PWM_4 -> /USB-
- J2 pad 23: /CAN_H -> /GPIO_5
- J2 pad 24: /CAN_L -> /GPIO_6
- J2 pad 25: /USB+ -> /GPIO_7
- J2 pad 26: /USB- -> /GPIO_8
- J4 pad 15: /PWM_2 -> /CAN_L
- J4 pad 16: /PWM_1 -> /CAN_H
- J4 pad 17: /PWM_4 -> /USB-
- J4 pad 18: /PWM_3 -> /USB+
- J4 pad 23: /CAN_L -> /GPIO_6
- J4 pad 24: /CAN_H -> /GPIO_5
- J4 pad 25: /USB- -> /GPIO_8
- J4 pad 26: /USB+ -> /GPIO_7
Routing:
- net /USB-: track 29.4 -> 23.9 mm
- net /USB+: track 36.3 -> 31.6 mm
- net Net-(D8-A): track 37.3 -> 38.8 mm
- net GND: vias 42 -> 47
- net /PWM_4: vias 2 -> 0
- net /PWM_3: vias 2 -> 0
- net /PWM_2: vias 2 -> 0
- net /PWM_1: vias 2 -> 0
- net /GPIO_8: vias 0 -> 2
- net /GPIO_7: vias 0 -> 2
- net /GPIO_6: vias 0 -> 2
- net /GPIO_5: vias 0 -> 2
