File: hw/kicad/base/12V/12V.kicad_sch (KiCad schematic)
At the start: 29 parts, among them J1 USB_B_Micro, J2 TOP, J3 XT60PW-M, J4 BUTTOM, U1 LM1117MP-3.3, U2 LM2596S-5, U3 CP2102N-Axx-xQFN28

Commit message: 修改尺寸至45x45
Parts:
- added D9: LED, LED_SMD:LED_0805_2012Metric, symbol Device:LED
- added JUMP1: 0, Resistor_SMD:R_01005_0402Metric, symbol Device:R
- added R5: 10k, Resistor_SMD:R_0805_2012Metric, symbol Device:R
- C1: footprint Capacitor_Tantalum_SMD:CP_EIA-3528-21_Kemet-B -> Capacitor_SMD:C_0805_2012Metric
- C10: value 10uF -> 47uF; footprint Capacitor_Tantalum_SMD:CP_EIA-3528-21_Kemet-B -> Capacitor_Tantalum_SMD:CP_EIA-3216-12_Kemet-S
- C2, C4, C5: footprint Capacitor_SMD:C_0603_1608Metric -> Capacitor_SMD:C_0805_2012Metric
- C6: footprint Capacitor_Tantalum_SMD:CP_EIA-3528-21_Kemet-B -> Capacitor_Tantalum_SMD:CP_EIA-6032-28_Kemet-C
- C9: value 10uF -> 0.1uF; footprint Capacitor_Tantalum_SMD:CP_EIA-3528-21_Kemet-B -> Capacitor_SMD:C_0805_2012Metric
- J1: footprint Connector_USB:USB_Micro-B_Molex_47346-0001 -> Connector_USB:USB_Micro-B_Wuerth_629105150521
- J3: value XT60PW-M -> XT30PW-M; footprint XT:XT60-PW-M -> XT:XT30-PAD
- R1, R2, R3, R4: footprint Resistor_SMD:R_0201_0603Metric -> Resistor_SMD:R_0805_2012Metric
Connections:
- net +3.3V: now also D9.2 (A)
- net +BATT: now also J3.2 (-); no longer J3.1 (+)
- net GND: now also J3.1 (+), R5.1; no longer J3.2 (-)
- net VBUS: now also JUMP1.1; no longer C4.2, U3.7 (VREGIN), U3.8 (VBUS)
- new net: C4.2, JUMP1.2, U3.7 (VREGIN), U3.8 (VBUS)
- new net: D9.1 (K), R5.2
Other:
- moved on the sheet: D7, D8

Commit message: 第二次打样的整改；dc motor改成了三路 io不够做不了四路；
Parts:
- JUMP1: footprint Resistor_SMD:R_01005_0402Metric -> Resistor_SMD:R_0603_1608Metric
Changed lines of the file:
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@@
       (effects (font (size 1.27 1.27)))
     )
-    (property "Footprint" "Resistor_SMD:R_01005_0402Metric" (at 109.855 51.943 90)
+    (property "Footprint" "Resistor_SMD:R_0603_1608Metric" (at 109.855 51.943 90)
       (effects (font (size 1.27 1.27)) hide)
     )

Commit message: 更换接口线序
Connections:
- net PWM_1 is gone; now on net CAN_H: J2.15 (Pin_15), J4.16 (Pin_16)
- net PWM_2 is gone; now on net CAN_L: J2.16 (Pin_16), J4.15 (Pin_15)
- net PWM_3 is gone; now on net USB+: J2.17 (Pin_17), J4.18 (Pin_18)
- net PWM_4 is gone; now on net USB-: J2.18 (Pin_18), J4.17 (Pin_17)
- net CAN_H: no longer J2.23 (Pin_23), J4.24 (Pin_24)
- net CAN_L: no longer J2.24 (Pin_24), J4.23 (Pin_23)
- net USB+: no longer J2.25 (Pin_25), J4.26 (Pin_26)
- net USB-: no longer J2.26 (Pin_26), J4.25 (Pin_25)
- net PWM_5 renamed GPIO_1
- net PWM_6 renamed GPIO_2
- net PWM_7 renamed GPIO_3
- net PWM_8 renamed GPIO_4
- new net GPIO_5: J2.23 (Pin_23), J4.24 (Pin_24)
- new net GPIO_6: J2.24 (Pin_24), J4.23 (Pin_23)
- new net GPIO_7: J2.25 (Pin_25), J4.26 (Pin_26)
- new net GPIO_8: J2.26 (Pin_26), J4.25 (Pin_25)
Changed lines of the file:
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@@
     (effects (font (size 1.27 1.27)) (justify left bottom))
   )
-  (label "PWM_5" (at 240.919 63.881 0) (fields_autoplaced)
-    (effects (font (size 1.27 1.27)) (justify left bottom))
-  )
-  (label "PWM_3" (at 240.919 61.341 0) (fields_autoplaced)
+  (label "GPIO_5" (at 240.919 68.961 0) (fields_autoplaced)
+    (effects (font (size 1.27 1.27)) (justify left bottom))
+  )
+  (label "GPIO_3" (at 240.919 66.421 0) (fields_autoplaced)
     (effects (font (size 1.27 1.27)) (justify left bottom))
   )
@@
     (effects (font (size 1.27 1.27)) (justify left bottom))
   )
-  (label "CAN_H" (at 240.919 68.961 0) (fields_autoplaced)
+  (label "CAN_H" (at 240.919 58.801 0) (fields_autoplaced)
     (effects (font (size 1.27 1.27)) (justify left bottom))
   )
@@
     (effects (font (size 1.27 1.27)) (justify right bottom))
   )
-  (label "PWM_4" (at 271.399 61.341 180) (fields_autoplaced)
-    (effects (font (size 1.27 1.27)) (justify right bottom))
-  )
-  (label "PWM_3" (at 205.74 61.468 0) (fields_autoplaced)
+  (label "GPIO_4" (at 271.399 66.421 180) (fields_autoplaced)
+    (effects (font (size 1.27 1.27)) (justify right bottom))
+  )
+  (label "GPIO_3" (at 205.74 66.548 0) (fields_autoplaced)
     (effects (font (size 1.27 1.27)) (justify left bottom))
   )
@@
     (effects (font (size 1.27 1.27)) (justify left bottom))
   )
-  (label "PWM_6" (at 271.399 63.881 180) (fields_autoplaced)
+  (label "GPIO_6" (at 271.399 68.961 180) (fields_autoplaced)
     (effects (font (size 1.27 1.27)) (justify right bottom))
   )
@@
     (effects (font (size 1.27 1.27)) (justify left bottom))
   )
-  (label "CAN_L" (at 236.22 69.088 180) (fields_autoplaced)
-    (effects (font (size 1.27 1.27)) (justify right bottom))
-  )
-  (label "PWM_1" (at 240.919 58.801 0) (fields_autoplaced)
-    (effects (font (size 1.27 1.27)) (justify left bottom))
-  )
-  (label "PWM_2" (at 271.399 58.801 180) (fields_autoplaced)
+  (label "CAN_L" (at 236.22 58.928 180) (fields_autoplaced)
+    (effects (font (size 1.27 1.27)) (justify right bottom))
+  )
+  (label "GPIO_1" (at 240.919 63.881 0) (fields_autoplaced)
+    (effects (font (size 1.27 1.27)) (justify left bottom))
+  )
+  (label "GPIO_2" (at 271.399 63.881 180) (fields_autoplaced)
     (effects (font (size 1.27 1.27)) (justify right bottom))
   )
@@
     (effects (font (size 1.27 1.27)) (justify right bottom))
   )
-  (label "PWM_7" (at 240.919 66.421 0) (fields_autoplaced)
-    (effects (font (size 1.27 1.27)) (justify left bottom))
-  )
-  (label "PWM_8" (at 236.22 66.548 180) (fields_autoplaced)
+  (label "GPIO_7" (at 240.919 71.501 0) (fields_autoplaced)
+    (effects (font (size 1.27 1.27)) (justify left bottom))
+  )
+  (label "GPIO_8" (at 236.22 71.628 180) (fields_autoplaced)
     (effects (font (size 1.27 1.27)) (justify right bottom))
   )
@@
     (effects (font (size 1.27 1.27)) (justify left bottom))
   )
-  (label "USB-" (at 271.399 71.501 180) (fields_autoplaced)
-    (effects (font (size 1.27 1.27)) (justify right bottom))
-  )
-  (label "PWM_7" (at 205.74 66.548 0) (fields_autoplaced)
+  (label "USB-" (at 271.399 61.341 180) (fields_autoplaced)
+    (effects (font (size 1.27 1.27)) (justify right bottom))
+  )
+  (label "GPIO_7" (at 205.74 71.628 0) (fields_autoplaced)
     (effects (font (size 1.27 1.27)) (justify left bottom))
   )
@@
     (effects (font (size 1.27 1.27)) (justify left bottom))
   )
-  (label "CAN_L" (at 271.399 68.961 180) (fields_autoplaced)
+  (label "CAN_L" (at 271.399 58.801 180) (fields_autoplaced)
     (effects (font (size 1.27 1.27)) (justify right bottom))
   )
@@
     (effects (font (size 1.27 1.27)) (justify right bottom))
   )
-  (label "CAN_H" (at 205.74 69.088 0) (fields_autoplaced)
+  (label "CAN_H" (at 205.74 58.928 0) (fields_autoplaced)
     (effects (font (size 1.27 1.27)) (justify left bottom))
   )
@@
     (effects (font (size 1.27 1.27)) (justify right bottom))
   )
-  (label "USB-" (at 236.22 71.628 180) (fields_autoplaced)
-    (effects (font (size 1.27 1.27)) (justify right bottom))
-  )
-  (label "PWM_6" (at 236.22 64.008 180) (fields_autoplaced)
+  (label "USB-" (at 236.22 61.468 180) (fields_autoplaced)
+    (effects (font (size 1.27 1.27)) (justify right bottom))
+  )
+  (label "GPIO_6" (at 236.22 69.088 180) (fields_autoplaced)
     (effects (font (size 1.27 1.27)) (justify right bottom))
   )
@@
     (effects (font (size 1.27 1.27)) (justify right bottom))
   )
-  (label "PWM_5" (at 205.74 64.008 0) (fields_autoplaced)
-    (effects (font (size 1.27 1.27)) (justify left bottom))
-  )
-  (label "PWM_4" (at 236.22 61.468 180) (fields_autoplaced)
-    (effects (font (size 1.27 1.27)) (justify right bottom))
-  )
-  (label "PWM_1" (at 205.74 58.928 0) (fields_autoplaced)
-    (effects (font (size 1.27 1.27)) (justify left bottom))
-  )
-  (label "USB+" (at 205.74 71.628 0) (fields_autoplaced)
+  (label "GPIO_5" (at 205.74 69.088 0) (fields_autoplaced)
+    (effects (font (size 1.27 1.27)) (justify left bottom))
+  )
+  (label "GPIO_4" (at 236.22 66.548 180) (fields_autoplaced)
+    (effects (font (size 1.27 1.27)) (justify right bottom))
+  )
+  (label "GPIO_1" (at 205.74 64.008 0) (fields_autoplaced)
+    (effects (font (size 1.27 1.27)) (justify left bottom))
+  )
+  (label "USB+" (at 205.74 61.468 0) (fields_autoplaced)
     (effects (font (size 1.27 1.27)) (justify left bottom))
   )
@@
     (effects (font (size 1.27 1.27)) (justify right bottom))
   )
-  (label "PWM_2" (at 236.22 58.928 180) (fields_autoplaced)
+  (label "GPIO_2" (at 236.22 64.008 180) (fields_autoplaced)
     (effects (font (size 1.27 1.27)) (justify right bottom))
   )
@@
     (effects (font (size 1.27 1.27)) (justify right bottom))
   )
-  (label "USB+" (at 240.919 71.501 0) (fields_autoplaced)
+  (label "USB+" (at 240.919 61.341 0) (fields_autoplaced)
     (effects (font (size 1.27 1.27)) (justify left bottom))
   )
@@
     (effects (font (size 1.27 1.27)) (justify right bottom))
   )
-  (label "PWM_8" (at 271.399 66.421 180) (fields_autoplaced)
-    (effects (font (size 1.27 1.27)) (justify right bottom))
-  )
+  (label "GPIO_8" (at 271.399 71.501 180) (fields_autoplaced)
+    (effects (font (size 1.27 1.27)) (justify right bottom))
+  )
