File: hw/kicad/cpu/esp32_wroom_32e/esp32_wroom_32e.kicad_pcb (KiCad board)
At the start: 2 copper layers, 50 x 50 mm, 30 parts, among them J1 Conn_02x20_Odd_Even, J2 Conn_02x20_Odd_Even, U1 ESP32-WROOM-32, U2 ICM-42688-P

Commit message: 更新了template
Parts:
- added D1: LED, LED_SMD:LED_0805_2012Metric, F.Cu at (104.7, 53.0)
- added R10: 10k, Resistor_SMD:R_0805_2012Metric, F.Cu at (106.9, 50.0)
- C1: value 200uF -> 47uF; footprint Capacitor_Tantalum_SMD:CP_EIA-7343-20_Kemet-V -> Capacitor_Tantalum_SMD:CP_EIA-3216-12_Kemet-S
- C2, C3, C4: footprint Capacitor_SMD:C_0603_1608Metric -> Capacitor_SMD:C_0805_2012Metric
- R7, R8: footprint Resistor_SMD:R_0603_1608Metric -> Resistor_SMD:R_0805_2012Metric
- moved R25 34.3 mm to (50.9, 59.5)
- moved R24 34.2 mm to (50.9, 63.4)
- moved R23 33.9 mm to (49.0, 59.5)
- moved R22 33.9 mm to (49.0, 63.4)
- moved R21 33.6 mm to (47.0, 59.5)
- moved R20 33.6 mm to (47.0, 63.4)
- moved R19 33.3 mm to (45.1, 59.5)
- moved R2 33.3 mm to (45.1, 63.4)
- moved R7 33.3 mm to (114.8, 53.0), turned to 0 degrees
- moved R8 33.0 mm to (114.8, 56.0), turned to 0 degrees
- moved R17 33.0 mm to (43.1, 59.5)
- moved R16 33.0 mm to (43.2, 63.4)
- moved R15 32.7 mm to (41.2, 59.5)
- moved R14 32.7 mm to (41.2, 63.4)
- moved R13 32.4 mm to (39.3, 59.5)
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Connections:
- U1 pad 24: /IMU_INT1 -> /LED
- U2 pad 4: /IMU_INT1 -> unconnected-(U2-INT1/INT-Pad4)
Routing:
- net +3.3V: track 90.7 -> 7.94 mm
- net /pwm7: track 58.7 -> 0.00 mm, vias 2 -> 0
- net /pwm8: track 51.0 -> 0.00 mm, vias 2 -> 0
- net /pwm5: track 48.8 -> 0.00 mm, vias 2 -> 0
- net /pwm3: track 43.3 -> 0.00 mm, vias 2 -> 0
- net /pwm6: track 41.7 -> 0.00 mm, vias 2 -> 0
- net /vspi_mosi: track 40.6 -> 0.00 mm, vias 2 -> 0
- net /uart0rx: track 31.3 -> 0.00 mm, vias 2 -> 0
- net /vspi_cs: track 29.4 -> 0.00 mm, vias 2 -> 0
- net /vspi_miso: track 28.6 -> 0.00 mm, vias 2 -> 0
- net /uart0tx: track 26.8 -> 0.00 mm, vias 2 -> 0
- net /vspi1_clk: track 25.0 -> 0.00 mm, vias 2 -> 0
- net /i2c_data: track 23.0 -> 0.00 mm, vias 2 -> 0
- net /i2c_clock: track 19.9 -> 0.00 mm, vias 2 -> 0
- net /IMU_INT1: track 17.3 -> 0.00 mm, vias 2 -> 0
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- removed copper zone on B.Cu, net GND
- removed copper zone on F.Cu, net GND
Other:
- board size 50 x 50 mm -> 45 x 45 mm

Commit message: Pindar v1.0
Parts:
- moved R8 52.5 mm to (62.2, 56.4), turned to -90 degrees
- moved R7 50.2 mm to (64.7, 56.4), turned to -90 degrees
- moved R17 48.3 mm to (91.4, 61.3)
- moved R16 48.3 mm to (91.4, 64.8)
- moved R15 47.8 mm to (88.9, 61.3)
- moved R14 47.7 mm to (88.9, 64.7)
- moved R24 45.8 mm to (96.3, 56.9)
- moved R25 45.8 mm to (96.3, 53.1)
- moved R22 45.3 mm to (93.9, 56.9)
- moved R23 45.3 mm to (93.8, 53.1)
- moved R20 44.8 mm to (91.4, 56.9)
- moved R21 44.8 mm to (91.4, 53.1)
- moved R19 44.3 mm to (88.9, 53.1)
- moved R2 44.3 mm to (88.9, 56.9)
- moved C4 36.6 mm to (71.8, 66.4), turned to 90 degrees
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Connections:
- net /vspi1_clk renamed /vspi_clk
- R1 pad 1: /adc1_ch3 -> /adc1_ch0
- R3 pad 1: /adc1_ch7 -> /adc1_ch6
- R4 pad 1: /adc1_ch6 -> /adc1_ch7
- R7 pad 2: /i2c_data -> /i2c_clock
- R8 pad 2: /i2c_clock -> /i2c_data
- R9 pad 1: /adc1_ch0 -> /adc1_ch3
- U1 pad 10: /pwm2 -> /pwm6
- U1 pad 11: /pwm1 -> /pwm4
- U1 pad 12: /pwm4 -> /pwm2
- U1 pad 26: /pwm3 -> /pwm1
- U1 pad 27: /pwm6 -> /pwm3
- U1 pad 8: /i2c_clock -> /i2c_data
- U1 pad 9: /i2c_data -> /i2c_clock
Routing:
- net +3.3V: track 7.94 -> 69.0 mm, vias 4 -> 10
- net /uart0rx: track 0.00 -> 38.1 mm, vias 0 -> 2
- net /PWM_2: track 2.98 -> 40.5 mm
- net /PWM_4: track 2.74 -> 38.8 mm
- net /PWM_8: track 2.69 -> 37.4 mm
- net /PWM_6: track 3.02 -> 37.0 mm
- net /PWM_1: track 7.59 -> 41.1 mm
- net /uart0tx: track 0.00 -> 33.3 mm, vias 0 -> 2
- net /PWM_3: track 7.45 -> 39.0 mm
- net /PWM_5: track 7.66 -> 37.5 mm
- net /PWM_7: track 7.60 -> 37.4 mm
- net /pwm6: track 0.00 -> 28.6 mm, vias 0 -> 2
- net /SPI_MISO: track 2.84 -> 30.6 mm
- net /pwm4: track 0.00 -> 26.2 mm, vias 0 -> 2
- net /SPI_CLK: track 3.01 -> 28.9 mm
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- added copper zone on B.Cu, net GND
- added copper zone on F.Cu, net GND
Other:
- board text added: "Pindar v1.0 Type CPU esp32 wroom 32e v1.0"

Commit message: 更换接口线序
Connections:
- J1 pad 15: /PWM_2 -> /CAN_L
- J1 pad 16: /PWM_1 -> /CAN_H
- J1 pad 17: /PWM_4 -> /USB-
- J1 pad 18: /PWM_3 -> /USB+
- J1 pad 19: /PWM_6 -> /PWM_2
- J1 pad 20: /PWM_5 -> /PWM_1
- J1 pad 21: /PWM_8 -> /PWM_4
- J1 pad 22: /PWM_7 -> /PWM_3
- J1 pad 23: /CAN_L -> /PWM_6
- J1 pad 24: /CAN_H -> /PWM_5
- J1 pad 25: /USB- -> /PWM_8
- J1 pad 26: /USB+ -> /PWM_7
- J2 pad 15: /PWM_1 -> /CAN_H
- J2 pad 16: /PWM_2 -> /CAN_L
- J2 pad 17: /PWM_3 -> /USB+
- J2 pad 18: /PWM_4 -> /USB-
- J2 pad 19: /PWM_5 -> /PWM_1
- J2 pad 20: /PWM_6 -> /PWM_2
- J2 pad 21: /PWM_7 -> /PWM_3
- J2 pad 22: /PWM_8 -> /PWM_4
- J2 pad 23: /CAN_H -> /PWM_5
- J2 pad 24: /CAN_L -> /PWM_6
- J2 pad 25: /USB+ -> /PWM_7
- J2 pad 26: /USB- -> /PWM_8
Routing:
- net /PWM_4: track 38.8 -> 35.8 mm
- net /PWM_3: track 39.0 -> 36.2 mm
- net /PWM_2: track 40.5 -> 37.8 mm
- net /PWM_1: track 41.1 -> 38.5 mm
- net /PWM_8: track 37.4 -> 34.9 mm
- net /PWM_6: track 37.0 -> 34.6 mm
- net /PWM_7: track 37.4 -> 35.0 mm
- net /PWM_5: track 37.5 -> 35.8 mm
- net /UART1_TX: track 15.1 -> 14.1 mm
- net /UART1_RX: track 14.8 -> 14.1 mm
- net GND: vias 53 -> 59
