File: hw/kicad/cpu/esp32_wroom_32e/esp32_wroom_32e.kicad_sch (KiCad schematic)
At the start: 30 parts, among them J1 Conn_02x20_Odd_Even, J2 Conn_02x20_Odd_Even, U1 ESP32-WROOM-32, U2 ICM-42688-P

Commit message: 更新了template
Parts:
- added D1: LED, LED_SMD:LED_0805_2012Metric, symbol Device:LED
- added R10: 10k, Resistor_SMD:R_0805_2012Metric, symbol Device:R
- C1: value 200uF -> 47uF; footprint Capacitor_Tantalum_SMD:CP_EIA-7343-20_Kemet-V -> Capacitor_Tantalum_SMD:CP_EIA-3216-12_Kemet-S
- C2, C3, C4: footprint Capacitor_SMD:C_0603_1608Metric -> Capacitor_SMD:C_0805_2012Metric
- R7, R8: footprint Resistor_SMD:R_0603_1608Metric -> Resistor_SMD:R_0805_2012Metric
Connections:
- net GND: now also R10.1
- net IMU_INT1: no longer names the net of U2.4 (INT1/INT)
- net IMU_INT1: no longer U1.24 (IO2)
- new net: D1.1 (K), R10.2
- new net LED: D1.2 (A), U1.24 (IO2)
- no-connect marks 6 -> 7
Changed lines of the file:
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@@
   (no_connect (at 52.705 139.065))
   (no_connect (at 52.705 131.445))
+  (no_connect (at 248.92 127))
   (no_connect (at 52.705 141.605))
   (no_connect (at 52.705 133.985))
@@
     (stroke (width 0) (type default))
   )
-  (wire (pts (xy 83.185 103.505) (xy 94.107 103.505))
+  (wire (pts (xy 83.185 103.505) (xy 91.948 103.505))
     (stroke (width 0) (type default))
   )
@@
     (stroke (width 0) (type default))
   )
+  (wire (pts (xy 159.893 130.175) (xy 165.354 130.175))
+    (stroke (width 0) (type default))
+  )
   (wire (pts (xy 135.255 39.37) (xy 149.86 39.37))
     (stroke (width 0) (type default))
@@
     (stroke (width 0) (type default))
   )
-  (wire (pts (xy 248.92 127) (xy 256.54 127))
-    (stroke (width 0) (type default))
-  )
   (wire (pts (xy 52.705 98.425) (xy 50.165 98.425))
     (stroke (width 0) (type default))
@@
     (stroke (width 0) (type default))
   )
+  (wire (pts (xy 144.399 133.35) (xy 144.399 130.175))
+    (stroke (width 0) (type default))
+  )
   (wire (pts (xy 253.365 115.57) (xy 253.365 119.38))
     (stroke (width 0) (type default))
@@
     (stroke (width 0) (type default))
   )
+  (wire (pts (xy 143.891 122.555) (xy 150.876 122.555))
+    (stroke (width 0) (type default))
+  )
   (wire (pts (xy 277.114 45.593) (xy 268.224 45.593))
     (stroke (width 0) (type default))
@@
     (stroke (width 0) (type default))
   )
+  (wire (pts (xy 158.496 122.555) (xy 165.354 122.555))
+    (stroke (width 0) (type default))
+  )
   (wire (pts (xy 246.634 88.773) (xy 255.524 88.773))
     (stroke (width 0) (type default))
@@
     (stroke (width 0) (type default))
   )
+  (wire (pts (xy 144.399 130.175) (xy 152.273 130.175))
+    (stroke (width 0) (type default))
+  )
   (wire (pts (xy 96.52 50.8) (xy 96.52 52.705))
     (stroke (width 0) (type default))
@@
     (stroke (width 0) (type default))
   )
+  (wire (pts (xy 165.354 122.555) (xy 165.354 130.175))
+    (stroke (width 0) (type default))
+  )
   (wire (pts (xy 83.185 128.905) (xy 93.98 128.905))
     (stroke (width 0) (type default))
@@
     (effects (font (size 1.27 1.27)) (justify right bottom))
   )
-  (label "IMU_INT1" (at 256.54 127 180) (fields_autoplaced)
-    (effects (font (size 1.27 1.27)) (justify right bottom))
-  )
   (label "PWM_2" (at 277.114 60.833 180) (fields_autoplaced)
     (effects (font (size 1.27 1.27)) (justify right bottom))
@@
     (effects (font (size 1.27 1.27)) (justify right bottom))
   )
-  (label "IMU_INT1" (at 94.107 103.505 180) (fields_autoplaced)
+  (label "LED" (at 91.948 103.505 180) (fields_autoplaced)
     (effects (font (size 1.27 1.27)) (justify right bottom))
   )
@@
   (label "PWM_5" (at 185.42 88.9 180) (fields_autoplaced)
     (effects (font (size 1.27 1.27)) (justify right bottom))
+  )
+  (label "LED" (at 143.891 122.555 0) (fields_autoplaced)
+    (effects (font (size 1.27 1.27)) (justify left bottom))
   )
   (label "I2C_SDA" (at 246.634 53.213 0) (fields_autoplaced)
@@
       (effects (font (size 1.27 1.27)) (justify left))
     )
-    (property "Footprint" "Capacitor_SMD:C_0603_1608Metric" (at 72.7202 60.325 0)
+    (property "Footprint" "Capacitor_SMD:C_0805_2012Metric" (at 72.7202 60.325 0)
       (effects (font (size 1.27 1.27)) hide)
     )
@@
       (effects (font (size 1.27 1.27)) (justify left))
     )
-    (property "Footprint" "Resistor_SMD:R_0603_1608Metric" (at 107.442 139.7 90)
+    (property "Footprint" "Resistor_SMD:R_0805_2012Metric" (at 107.442 139.7 90)
       (effects (font (size 1.27 1.27)) hide)
     )
@@
       (effects (font (size 1.27 1.27)) (justify left))
     )
-    (property "Footprint" "Resistor_SMD:R_0603_1608Metric" (at 104.267 143.51 90)
+    (property "Footprint" "Resistor_SMD:R_0805_2012Metric" (at 104.267 143.51 90)
       (effects (font (size 1.27 1.27)) hide)
     )
@@
         (path "/988ee502-8596-4ebe-9b99-0eb76e7d156a"
           (reference "R3") (unit 1)
-        )
-      )
-    )
-  )
-  (symbol (lib_id "Device:C") (at 57.15 56.515 0) (unit 1)
-    (in_bom yes) (on_board yes) (dnp no) (fields_autoplaced)
-    (property "Reference" "C1" (at 60.96 55.245 0)
-      (effects (font (size 1.27 1.27)) (justify left))
-    )
-    (property "Value" "200uF" (at 60.96 57.785 0)
-      (effects (font (size 1.27 1.27)) (justify left))
-    )
-    (property "Footprint" "Capacitor_Tantalum_SMD:CP_EIA-7343-20_Kemet-V" (at 58.1152 60.325 0)
-      (effects (font (size 1.27 1.27)) hide)
-    )
-    (property "Datasheet" "~" (at 57.15 56.515 0)
-      (effects (font (size 1.27 1.27)) hide)
-    )
-    (pin "1")
-    (pin "2")
-    (instances
-      (project "esp32_wroom_32e"
-        (path "/988ee502-8596-4ebe-9b99-0eb76e7d156a"
-          (reference "C1") (unit 1)
         )
       )
@@
     )
   )
+  (symbol (lib_id "Device:R") (at 156.083 130.175 90) (unit 1)
+    (in_bom yes) (on_board yes) (dnp no)
+    (property "Reference" "R10" (at 157.861 128.016 90)
+      (effects (font (size 1.27 1.27)) (justify left))
+    )
+    (property "Value" "10k" (at 158.115 132.207 90)
+      (effects (font (size 1.27 1.27)) (justify left))
+    )
+    (property "Footprint" "Resistor_SMD:R_0805_2012Metric" (at 156.083 131.953 90)
+      (effects (font (size 1.27 1.27)) hide)
+    )
+    (property "Datasheet" "~" (at 156.083 130.175 0)
+      (effects (font (size 1.27 1.27)) hide)
+    )
+    (pin "1")
+    (pin "2")
+    (instances
+      (project "esp32_wroom_32e"
+        (path "/988ee502-8596-4ebe-9b99-0eb76e7d156a"
+          (reference "R10") (unit 1)
+        )
+      )
+    )
+  )
   (symbol (lib_id "Connector_Generic:Conn_02x20_Odd_Even") (at 225.425 66.04 0) (unit 1)
     (in_bom yes) (on_board yes) (dnp no) (fields_autoplaced)
@@
       (effects (font (size 1.27 1.27)) (justify left))
     )
-    (property "Footprint" "Capacitor_SMD:C_0603_1608Metric" (at 97.4852 60.325 0)
+    (property "Footprint" "Capacitor_SMD:C_0805_2012Metric" (at 97.4852 60.325 0)
       (effects (font (size 1.27 1.27)) hide)
     )
@@
         (path "/988ee502-8596-4ebe-9b99-0eb76e7d156a"
           (reference "R21") (unit 1)
+        )
+      )
+    )
+  )
+  (symbol (lib_id "power:GND") (at 144.399 133.35 0) (unit 1)
+    (in_bom yes) (on_board yes) (dnp no) (fields_autoplaced)
+    (property "Reference" "#PWR03" (at 144.399 139.7 0)
+      (effects (font (size 1.27 1.27)) hide)
+    )
+    (property "Value" "GND" (at 144.399 137.795 0)
+      (effects (font (size 1.27 1.27)))
+    )
+    (property "Footprint" "" (at 144.399 133.35 0)
+      (effects (font (size 1.27 1.27)) hide)
+    )
+    (property "Datasheet" "" (at 144.399 133.35 0)
+      (effects (font (size 1.27 1.27)) hide)
+    )
+    (pin "1")
+    (instances
+      (project "esp32_wroom_32e"
+        (path "/988ee502-8596-4ebe-9b99-0eb76e7d156a"
+          (reference "#PWR03") (unit 1)
         )
       )
@@
       (effects (font (size 1.27 1.27)) (justify left))
     )
-    (property "Footprint" "Capacitor_SMD:C_0603_1608Metric" (at 84.7852 60.325 0)
+    (property "Footprint" "Capacitor_SMD:C_0805_2012Metric" (at 84.7852 60.325 0)
       (effects (font (size 1.27 1.27)) hide)
     )
@@
         )
       )
+    )
+  )
+  (symbol (lib_id "Device:C") (at 57.15 56.515 0) (unit 1)
+    (in_bom yes) (on_board yes) (dnp no) (fields_autoplaced)
+    (property "Reference" "C1" (at 60.325 55.245 0)
+      (effects (font (size 1.27 1.27)) (justify left))
+    )
+    (property "Value" "47uF" (at 60.325 57.785 0)
+      (effects (font (size 1.27 1.27)) (justify left))
+    )
+    (property "Footprint" "Capacitor_Tantalum_SMD:CP_EIA-3216-12_Kemet-S" (at 58.1152 60.325 0)
+      (effects (font (size 1.27 1.27)))
+    )
+    (property "Datasheet" "~" (at 57.15 56.515 0)
+      (effects (font (size 1.27 1.27)) hide)
+    )
+    (pin "1")
+    (pin "2")
+    (instances
+      (project "esp32_wroom_32e"
+        (path "/988ee502-8596-4ebe-9b99-0eb76e7d156a"
+          (reference "C1") (unit 1)
+        )
+      )
+    )
+  )
+  (symbol (lib_id "Device:LED") (at 154.686 122.555 180) (unit 1)
+    (in_bom yes) (on_board yes) (dnp no) (fields_autoplaced)
+    (property "Reference" "D1" (at 156.2735 115.5953 0)
+      (effects (font (size 1.27 1.27)))
+    )
+    (property "Value" "LED" (at 156.2735 118.1353 0)
+      (effects (font (size 1.27 1.27)))
+    )
+    (property "Footprint" "LED_SMD:LED_0805_2012Metric" (at 154.686 122.555 0)
+      (effects (font (size 1.27 1.27)) hide)
+    )
+    (property "Datasheet" "~" (at 154.686 122.555 0)
+      (effects (font (size 1.27 1.27)) hide)
+    )
+    (pin "1")
+    (pin "2")
+    (instances
+      (project "esp32_wroom_32e"
+        (path "/988ee502-8596-4ebe-9b99-0eb76e7d156a"
+          (reference "D1") (unit 1)
+        )
+      )

Commit message: Pindar v1.0
Connections:
- net adc1_ch0: now also R1.1; no longer R9.1
- net adc1_ch3: now also R9.1; no longer R1.1
- net adc1_ch6: now also R3.1; no longer R4.1
- net adc1_ch7: now also R4.1; no longer R3.1
- net i2c_clock: now also R7.2, U1.9 (IO33); no longer R8.2, U1.8 (IO32)
- net i2c_data: now also R8.2, U1.8 (IO32); no longer R7.2, U1.9 (IO33)
- net pwm1: now also U1.26 (IO4); no longer U1.11 (IO26)
- net pwm2: now also U1.12 (IO27); no longer U1.10 (IO25)
- net pwm3: now also U1.27 (IO16); no longer U1.26 (IO4)
- net pwm4: now also U1.11 (IO26); no longer U1.12 (IO27)
- net pwm6: now also U1.10 (IO25); no longer U1.27 (IO16)
- net vspi1_clk renamed vspi_clk
Changed lines of the file:
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@@
     (effects (font (size 1.27 1.27)) (justify left bottom))
   )
-  (label "adc1_ch3" (at 135.255 39.37 0) (fields_autoplaced)
+  (label "adc1_ch0" (at 135.255 39.37 0) (fields_autoplaced)
     (effects (font (size 1.27 1.27)) (justify left bottom))
   )
@@
     (effects (font (size 1.27 1.27)) (justify right bottom))
   )
-  (label "adc1_ch6" (at 135.255 46.99 0) (fields_autoplaced)
+  (label "adc1_ch7" (at 135.255 46.99 0) (fields_autoplaced)
     (effects (font (size 1.27 1.27)) (justify left bottom))
   )
@@
     (effects (font (size 1.27 1.27)) (justify right bottom))
   )
-  (label "pwm2" (at 92.71 141.605 180) (fields_autoplaced)
+  (label "pwm6" (at 92.71 141.605 180) (fields_autoplaced)
     (effects (font (size 1.27 1.27)) (justify right bottom))
   )
@@
     (effects (font (size 1.27 1.27)) (justify left bottom))
   )
-  (label "pwm1" (at 92.71 144.145 180) (fields_autoplaced)
+  (label "pwm4" (at 92.71 144.145 180) (fields_autoplaced)
     (effects (font (size 1.27 1.27)) (justify right bottom))
   )
@@
     (effects (font (size 1.27 1.27)) (justify right bottom))
   )
-  (label "adc1_ch0" (at 135.255 41.91 0) (fields_autoplaced)
+  (label "adc1_ch3" (at 135.255 41.91 0) (fields_autoplaced)
     (effects (font (size 1.27 1.27)) (justify left bottom))
   )
@@
     (effects (font (size 1.27 1.27)) (justify right bottom))
   )
-  (label "pwm4" (at 92.71 146.685 180) (fields_autoplaced)
+  (label "pwm2" (at 92.71 146.685 180) (fields_autoplaced)
     (effects (font (size 1.27 1.27)) (justify right bottom))
   )
@@
     (effects (font (size 1.27 1.27)) (justify right bottom))
   )
-  (label "vspi1_clk" (at 93.98 128.905 180) (fields_autoplaced)
+  (label "vspi_clk" (at 93.98 128.905 180) (fields_autoplaced)
     (effects (font (size 1.27 1.27)) (justify right bottom))
   )
@@
     (effects (font (size 1.27 1.27)) (justify right bottom))
   )
-  (label "i2c_data" (at 123.825 151.765 180) (fields_autoplaced)
+  (label "i2c_clock" (at 123.825 151.765 180) (fields_autoplaced)
     (effects (font (size 1.27 1.27)) (justify right bottom))
   )
@@
     (effects (font (size 1.27 1.27)) (justify right bottom))
   )
-  (label "i2c_clock" (at 117.856 149.098 180) (fields_autoplaced)
+  (label "i2c_data" (at 117.856 149.098 180) (fields_autoplaced)
     (effects (font (size 1.27 1.27)) (justify right bottom))
   )
@@
     (effects (font (size 1.27 1.27)) (justify right bottom))
   )
-  (label "pwm6" (at 93.98 123.825 180) (fields_autoplaced)
+  (label "pwm3" (at 93.98 123.825 180) (fields_autoplaced)
     (effects (font (size 1.27 1.27)) (justify right bottom))
   )
@@
     (effects (font (size 1.27 1.27)) (justify right bottom))
   )
-  (label "pwm3" (at 92.075 108.585 180) (fields_autoplaced)
+  (label "pwm1" (at 92.075 108.585 180) (fields_autoplaced)
     (effects (font (size 1.27 1.27)) (justify right bottom))
   )
@@
     (effects (font (size 1.27 1.27)) (justify left bottom))
   )
-  (label "vspi1_clk" (at 135.89 68.58 0) (fields_autoplaced)
+  (label "vspi_clk" (at 135.89 68.58 0) (fields_autoplaced)
     (effects (font (size 1.27 1.27)) (justify left bottom))
   )
@@
     (effects (font (size 1.27 1.27)) (justify right bottom))
   )
-  (label "adc1_ch7" (at 135.255 44.45 0) (fields_autoplaced)
-    (effects (font (size 1.27 1.27)) (justify left bottom))
-  )
+  (label "adc1_ch6" (at 135.255 44.45 0) (fields_autoplaced)
+    (effects (font (size 1.27 1.27)) (justify left bottom))
+  )

Commit message: 更换接口线序
Connections:
- net CAN_H: now also J1.16 (Pin_16), J2.15 (Pin_15); no longer J1.24 (Pin_24), J2.23 (Pin_23)
- net CAN_L: now also J1.15 (Pin_15), J2.16 (Pin_16); no longer J1.23 (Pin_23), J2.24 (Pin_24)
- net PWM_1: now also J1.20 (Pin_20), J2.19 (Pin_19); no longer J1.16 (Pin_16), J2.15 (Pin_15)
- net PWM_2: now also J1.19 (Pin_19), J2.20 (Pin_20); no longer J1.15 (Pin_15), J2.16 (Pin_16)
- net PWM_3: now also J1.22 (Pin_22), J2.21 (Pin_21); no longer J1.18 (Pin_18), J2.17 (Pin_17)
- net PWM_4: now also J1.21 (Pin_21), J2.22 (Pin_22); no longer J1.17 (Pin_17), J2.18 (Pin_18)
- net PWM_5: now also J1.24 (Pin_24), J2.23 (Pin_23); no longer J1.20 (Pin_20), J2.19 (Pin_19)
- net PWM_6: now also J1.23 (Pin_23), J2.24 (Pin_24); no longer J1.19 (Pin_19), J2.20 (Pin_20)
- net PWM_7: now also J1.26 (Pin_26), J2.25 (Pin_25); no longer J1.22 (Pin_22), J2.21 (Pin_21)
- net PWM_8: now also J1.25 (Pin_25), J2.26 (Pin_26); no longer J1.21 (Pin_21), J2.22 (Pin_22)
- net USB+: now also J1.18 (Pin_18), J2.17 (Pin_17); no longer J1.26 (Pin_26), J2.25 (Pin_25)
- net USB-: now also J1.17 (Pin_17), J2.18 (Pin_18); no longer J1.25 (Pin_25), J2.26 (Pin_26)
Changed lines of the file:
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@@
     (effects (font (size 1.27 1.27)) (justify right bottom))
   )
-  (label "PWM_7" (at 211.455 68.58 0) (fields_autoplaced)
+  (label "PWM_7" (at 211.455 73.66 0) (fields_autoplaced)
     (effects (font (size 1.27 1.27)) (justify left bottom))
   )
@@
     (effects (font (size 1.27 1.27)) (justify left bottom))
   )
-  (label "PWM_8" (at 277.114 68.453 180) (fields_autoplaced)
-    (effects (font (size 1.27 1.27)) (justify right bottom))
-  )
-  (label "PWM_1" (at 211.455 60.96 0) (fields_autoplaced)
-    (effects (font (size 1.27 1.27)) (justify left bottom))
-  )
-  (label "PWM_8" (at 241.935 68.58 180) (fields_autoplaced)
+  (label "PWM_8" (at 277.114 73.533 180) (fields_autoplaced)
+    (effects (font (size 1.27 1.27)) (justify right bottom))
+  )
+  (label "PWM_1" (at 211.455 66.04 0) (fields_autoplaced)
+    (effects (font (size 1.27 1.27)) (justify left bottom))
+  )
+  (label "PWM_8" (at 241.935 73.66 180) (fields_autoplaced)
     (effects (font (size 1.27 1.27)) (justify right bottom))
   )
@@
     (effects (font (size 1.27 1.27)) (justify left bottom))
   )
-  (label "USB+" (at 246.634 73.533 0) (fields_autoplaced)
+  (label "USB+" (at 246.634 63.373 0) (fields_autoplaced)
     (effects (font (size 1.27 1.27)) (justify left bottom))
   )
@@
     (effects (font (size 1.27 1.27)) (justify right bottom))
   )
-  (label "PWM_2" (at 277.114 60.833 180) (fields_autoplaced)
+  (label "PWM_2" (at 277.114 65.913 180) (fields_autoplaced)
     (effects (font (size 1.27 1.27)) (justify right bottom))
   )
@@
     (effects (font (size 1.27 1.27)) (justify left bottom))
   )
-  (label "PWM_6" (at 277.114 65.913 180) (fields_autoplaced)
+  (label "PWM_6" (at 277.114 70.993 180) (fields_autoplaced)
     (effects (font (size 1.27 1.27)) (justify right bottom))
   )
@@
     (effects (font (size 1.27 1.27)) (justify left bottom))
   )
-  (label "CAN_L" (at 277.114 70.993 180) (fields_autoplaced)
+  (label "CAN_L" (at 277.114 60.833 180) (fields_autoplaced)
     (effects (font (size 1.27 1.27)) (justify right bottom))
   )
@@
     (effects (font (size 1.27 1.27)) (justify left bottom))
   )
-  (label "CAN_L" (at 241.935 71.12 180) (fields_autoplaced)
+  (label "CAN_L" (at 241.935 60.96 180) (fields_autoplaced)
     (effects (font (size 1.27 1.27)) (justify right bottom))
   )
@@
     (effects (font (size 1.27 1.27)) (justify left bottom))
   )
-  (label "USB-" (at 277.114 73.533 180) (fields_autoplaced)
+  (label "USB-" (at 277.114 63.373 180) (fields_autoplaced)
     (effects (font (size 1.27 1.27)) (justify right bottom))
   )
@@
     (effects (font (size 1.27 1.27)) (justify right bottom))
   )
-  (label "PWM_6" (at 241.935 66.04 180) (fields_autoplaced)
+  (label "PWM_6" (at 241.935 71.12 180) (fields_autoplaced)
     (effects (font (size 1.27 1.27)) (justify right bottom))
   )
@@
     (effects (font (size 1.27 1.27)) (justify right bottom))
   )
-  (label "PWM_5" (at 211.455 66.04 0) (fields_autoplaced)
+  (label "PWM_5" (at 211.455 71.12 0) (fields_autoplaced)
     (effects (font (size 1.27 1.27)) (justify left bottom))
   )
@@
     (effects (font (size 1.27 1.27)) (justify left bottom))
   )
-  (label "PWM_7" (at 246.634 68.453 0) (fields_autoplaced)
+  (label "PWM_7" (at 246.634 73.533 0) (fields_autoplaced)
     (effects (font (size 1.27 1.27)) (justify left bottom))
   )
@@
     (effects (font (size 1.27 1.27)) (justify right bottom))
   )
-  (label "PWM_3" (at 246.634 63.373 0) (fields_autoplaced)
+  (label "PWM_3" (at 246.634 68.453 0) (fields_autoplaced)
     (effects (font (size 1.27 1.27)) (justify left bottom))
   )
@@
     (effects (font (size 1.27 1.27)) (justify right bottom))
   )
-  (label "PWM_1" (at 246.634 60.833 0) (fields_autoplaced)
+  (label "PWM_1" (at 246.634 65.913 0) (fields_autoplaced)
     (effects (font (size 1.27 1.27)) (justify left bottom))
   )
@@
     (effects (font (size 1.27 1.27)) (justify left bottom))
   )
-  (label "USB+" (at 211.455 73.66 0) (fields_autoplaced)
+  (label "USB+" (at 211.455 63.5 0) (fields_autoplaced)
     (effects (font (size 1.27 1.27)) (justify left bottom))
   )
@@
     (effects (font (size 1.27 1.27)) (justify right bottom))
   )
-  (label "PWM_2" (at 241.935 60.96 180) (fields_autoplaced)
+  (label "PWM_2" (at 241.935 66.04 180) (fields_autoplaced)
     (effects (font (size 1.27 1.27)) (justify right bottom))
   )
@@
     (effects (font (size 1.27 1.27)) (justify right bottom))
   )
-  (label "PWM_3" (at 211.455 63.5 0) (fields_autoplaced)
+  (label "PWM_3" (at 211.455 68.58 0) (fields_autoplaced)
     (effects (font (size 1.27 1.27)) (justify left bottom))
   )
@@
     (effects (font (size 1.27 1.27)) (justify left bottom))
   )
-  (label "CAN_H" (at 211.455 71.12 0) (fields_autoplaced)
+  (label "CAN_H" (at 211.455 60.96 0) (fields_autoplaced)
     (effects (font (size 1.27 1.27)) (justify left bottom))
   )
@@
     (effects (font (size 1.27 1.27)) (justify right bottom))
   )
-  (label "PWM_4" (at 277.114 63.373 180) (fields_autoplaced)
+  (label "PWM_4" (at 277.114 68.453 180) (fields_autoplaced)
     (effects (font (size 1.27 1.27)) (justify right bottom))
   )
@@
     (effects (font (size 1.27 1.27)) (justify right bottom))
   )
-  (label "USB-" (at 241.935 73.66 180) (fields_autoplaced)
-    (effects (font (size 1.27 1.27)) (justify right bottom))
-  )
-  (label "PWM_5" (at 246.634 65.913 0) (fields_autoplaced)
+  (label "USB-" (at 241.935 63.5 180) (fields_autoplaced)
+    (effects (font (size 1.27 1.27)) (justify right bottom))
+  )
+  (label "PWM_5" (at 246.634 70.993 0) (fields_autoplaced)
     (effects (font (size 1.27 1.27)) (justify left bottom))
   )
@@
     (effects (font (size 1.27 1.27)) (justify right bottom))
   )
-  (label "PWM_4" (at 241.935 63.5 180) (fields_autoplaced)
+  (label "PWM_4" (at 241.935 68.58 180) (fields_autoplaced)
     (effects (font (size 1.27 1.27)) (justify right bottom))
   )
@@
     (effects (font (size 1.27 1.27)) (justify right bottom))
   )
-  (label "CAN_H" (at 246.634 70.993 0) (fields_autoplaced)
-    (effects (font (size 1.27 1.27)) (justify left bottom))
-  )
+  (label "CAN_H" (at 246.634 60.833 0) (fields_autoplaced)
+    (effects (font (size 1.27 1.27)) (justify left bottom))
+  )
