File: hw/kicad/app/gyro/gyro.kicad_pcb (KiCad board)
At the start: 2 copper layers, 10 x 12 mm, 14 parts, among them U1 ICM-42688-P, U2 BMI088

Commit message: 更新app gyro板
Parts:
- removed the ? at (56.3, 59.6) (x2)
- removed the ? at (50.1, 59.6) (x2)
- removed the ? at (54.3, 59.6) (x2)
- removed the ? at (52.2, 59.6) (x2)
- added ?: , , F.Cu at (53.8, 60.3)
- added ?: , , F.Cu at (50.1, 60.3)
- added ?: , , F.Cu at (51.3, 60.3)
- added ?: , , F.Cu at (52.6, 60.3)
- added ?: , , F.Cu at (55.1, 60.3)
- added ?: , , F.Cu at (56.3, 60.3)
- added ?: , , B.Cu at (53.8, 60.4)
- added ?: , , B.Cu at (52.6, 60.3)
Connections:
- U2 pad 14: /spi_cs -> /IO2
Routing:
- net /IO2: track 0.00 -> 12.5 mm
- net /spi_cs: track 16.5 -> 5.81 mm, vias 1 -> 0
- net /spi_mosi: track 5.52 -> 6.34 mm
- net +3.3V: track 27.0 -> 26.2 mm
- net GND: vias 12 -> 8
Other:
- board size 10 x 12 mm -> 8.8 x 12 mm
