File: hw/kicad/app/gyro/gyro.kicad_sch (KiCad schematic)
At the start: 8 parts, among them J1 GHS-TBT(LF)(SN)(N), J2 GHS-TBT(LF)(SN)(N), U1 ICM-42688-P, U2 BMI088

Commit message: 更新app gyro板
Parts:
- J1: footprint (none) -> Connector_JST:JST_GH_SM06B-GHS-TB_1x06-1MP_P1.25mm_Horizontal
- J2: footprint (none) -> Connector_JST:JST_GH_SM04B-GHS-TB_1x04-1MP_P1.25mm_Horizontal
Connections:
- net spi_cs: no longer U2.14 (CSB1)
- net IO2: now reaches J2.3
- net IO2: now also U2.14 (CSB1)
- no-connect marks 7 -> 6
Changed lines of the file:
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@@
   (no_connect (at 214.249 83.693))
   (no_connect (at 80.264 112.903))
-  (no_connect (at 236.982 117.475))
   (no_connect (at 214.249 81.153))
   (wire (pts (xy 236.982 117.475) (xy 245.491 117.475))
@@
     (stroke (width 0) (type default))
   )
+  (wire (pts (xy 255.524 90.805) (xy 238.379 90.805))
+    (stroke (width 0) (type default))
+  )
   (wire (pts (xy 78.486 62.357) (xy 78.613 62.357))
     (stroke (width 0) (type default))
@@
     (stroke (width 0) (type default))
   )
-  (wire (pts (xy 238.379 90.805) (xy 257.429 90.805))
+  (wire (pts (xy 255.524 90.801) (xy 257.5805 90.801))
+    (stroke (width 0) (type default))
+  )
+  (wire (pts (xy 255.524 90.801) (xy 255.524 90.805))
     (stroke (width 0) (type default))
   )
@@
     (effects (font (size 1.27 1.27)) (justify left bottom))
   )
-  (label "spi_cs" (at 257.429 90.805 180) (fields_autoplaced)
+  (label "+3.3V" (at 183.642 110.871 0) (fields_autoplaced)
+    (effects (font (size 1.27 1.27)) (justify left bottom))
+  )
+  (label "spi_clk" (at 71.374 120.523 0) (fields_autoplaced)
+    (effects (font (size 1.27 1.27)) (justify left bottom))
+  )
+  (label "IO2" (at 257.5805 90.801 180) (fields_autoplaced)
     (effects (font (size 1.27 1.27)) (justify right bottom))
   )
-  (label "+3.3V" (at 183.642 110.871 0) (fields_autoplaced)
-    (effects (font (size 1.27 1.27)) (justify left bottom))
-  )
-  (label "spi_clk" (at 71.374 120.523 0) (fields_autoplaced)
-    (effects (font (size 1.27 1.27)) (justify left bottom))
-  )
   (label "spi_cs" (at 71.374 117.983 0) (fields_autoplaced)
     (effects (font (size 1.27 1.27)) (justify left bottom))
   )
   (label "spi_miso" (at 183.642 121.031 0) (fields_autoplaced)
+    (effects (font (size 1.27 1.27)) (justify left bottom))
+  )
+  (label "IO2" (at 236.982 117.475 0) (fields_autoplaced)
     (effects (font (size 1.27 1.27)) (justify left bottom))
   )
@@
       (effects (font (size 1.27 1.27)) (justify left))
     )
-    (property "Footprint" "" (at 255.651 117.475 0)
+    (property "Footprint" "Connector_JST:JST_GH_SM04B-GHS-TB_1x04-1MP_P1.25mm_Horizontal" (at 255.651 117.475 0)
       (effects (font (size 1.27 1.27)) (justify bottom) hide)
     )
@@
       (effects (font (size 1.27 1.27)) (justify left))
     )
-    (property "Footprint" "" (at 201.549 118.491 0)
-      (effects (font (size 1.27 1.27)) (justify bottom) hide)
-    )
+    (property "Footprint" "Connector_JST:JST_GH_SM06B-GHS-TB_1x06-1MP_P1.25mm_Horizontal" (at 201.549 118.491 0)
+      (effects (font (size 1.27 1.27)) (justify bottom) hide)
+    )
