File: hw/kicad/app/pmw3360/pmw3360.kicad_sch (KiCad schematic)
At the start: 13 parts, among them J2 TOP, J4 BUTTOM, U1 PMW3360DM-T2QU, U2 AMS1117-1.8

Commit message: 尽力改成40mmx40mm
Parts:
- removed J4: BUTTOM, Connector_PinHeader_1.27mm:PinHeader_2x20_P1.27mm_Vertical_SMD, symbol Connector_Generic:Conn_02x20_Odd_Even
- added J1: TOP, Connector_PinHeader_1.27mm:PinHeader_2x20_P1.27mm_Vertical_SMD, symbol Connector_Generic:Conn_02x20_Odd_Even
- J2: value TOP -> BUTTOM
Connections:
- net +3.3V: now also R1.2, J1.27 (Pin_27), J1.28 (Pin_28); no longer R1.1, U1.7 (~{RESET})
- net +5V: now also J1.29 (Pin_29), J1.30 (Pin_30)
- net +BATT: now also J1.33 (Pin_33), J1.34 (Pin_34), J1.35 (Pin_35), J1.36 (Pin_36)
- net ADC_1: now also J2.2 (Pin_2), J1.1 (Pin_1); no longer J2.1 (Pin_1)
- net ADC_2: now also J2.1 (Pin_1), J1.2 (Pin_2); no longer J2.2 (Pin_2)
- net ADC_3: now also J2.4 (Pin_4), J1.3 (Pin_3); no longer J2.3 (Pin_3)
- net ADC_4: now also J2.3 (Pin_3), J1.4 (Pin_4); no longer J2.4 (Pin_4)
- net GND: now also J1.31 (Pin_31), J1.32 (Pin_32), J1.37 (Pin_37), J1.38 (Pin_38), J1.39 (Pin_39), J1.40 (Pin_40)
- net I2C_CLK: now also J2.9 (Pin_9), J1.10 (Pin_10); no longer J2.10 (Pin_10)
- net I2C_SDA: now also J2.10 (Pin_10), J1.9 (Pin_9); no longer J2.9 (Pin_9)
- net SPI_CLK: now also J2.11 (Pin_11), J1.12 (Pin_12); no longer J2.12 (Pin_12)
- net SPI_CS: now also J2.12 (Pin_12), J1.11 (Pin_11); no longer J2.11 (Pin_11)
- net SPI_MISO: now also J2.13 (Pin_13), J1.14 (Pin_14); no longer J2.14 (Pin_14)
- net SPI_MOSI: now also J2.14 (Pin_14), J1.13 (Pin_13); no longer J2.13 (Pin_13)
- net at C2.1: now also R1.1, U1.7 (~{RESET}); no longer R1.2
- net CAN_H renamed GPIO_10
- net GPIO_10: now also J1.24 (Pin_24)
- net CAN_L: no longer names the net of U1.9 (MOTION)
- net CAN_L: no longer J2.24 (Pin_24)
- net PWM_1 renamed GPIO_2
- net GPIO_2: now also J1.16 (Pin_16)
- net PWM_2 renamed GPIO_1
- net GPIO_1: now also J1.15 (Pin_15)
- net PWM_3 renamed GPIO_4
- net GPIO_4: now also J1.18 (Pin_18)
- net PWM_4 renamed GPIO_3
- net GPIO_3: now also J1.17 (Pin_17)
- net PWM_5 renamed GPIO_6
- net GPIO_6: now also J1.20 (Pin_20)
- net PWM_6 renamed GPIO_5
- net GPIO_5: now also J1.19 (Pin_19)
- net PWM_7 renamed GPIO_8
- net GPIO_8: now also J1.22 (Pin_22)
- net PWM_8 renamed GPIO_7
- net GPIO_7: now also J1.21 (Pin_21)
- net UART1_RX renamed UART1_Tx
- net UART1_Tx: now also J1.6 (Pin_6)
- net UART1_TX renamed UART1_Rx
- net UART1_Rx: now also J1.5 (Pin_5)
- net UART2_RX renamed UART2_Tx
- net UART2_Tx: now also J1.8 (Pin_8)
- net UART2_TX renamed UART2_Rx
- net UART2_Rx: now also J1.7 (Pin_7)
- net USB+ renamed GPIO_12
- net GPIO_12: now also J1.26 (Pin_26)
- net USB- renamed GPIO_11
- net GPIO_11: now also J1.25 (Pin_25)
- new net GPIO_9: J1.23 (Pin_23), J2.24 (Pin_24)
- no-connect marks 0 -> 1
Other:
- moved on the sheet: C1, C2, C3, C4, C5, C6, R2, R3, U1, U2
