File: hw/kicad/cpu/esp32 s3/esp32 s3.kicad_pcb (KiCad board)
At the start: 2 copper layers, 40 x 40 mm, 18 parts, among them J1 TOP, J2 BUTTOM, J3 USB_B_Micro, SW1 SW_Push, SW2 SW_Push, U1 ESP32-S3-WROOM-1-N16R2, U2 ICM-42688-P

Commit message: cpu板io电阻
Parts:
- removed SW2: SW_Push, Button_Switch_THT:SW_SPST_Omron_B3F-315x_Angled
- added R10: R, Resistor_SMD:R_0603_1608Metric, F.Cu at (64.6, 64.4)
- added R11: R, Resistor_SMD:R_0603_1608Metric, F.Cu at (66.1, 64.4)
- added R12: R, Resistor_SMD:R_0603_1608Metric, F.Cu at (67.6, 64.4)
- added R13: R, Resistor_SMD:R_0603_1608Metric, F.Cu at (69.1, 64.4)
- added R14: R, Resistor_SMD:R_0603_1608Metric, F.Cu at (70.6, 64.4)
- added R15: R, Resistor_SMD:R_0603_1608Metric, F.Cu at (72.1, 64.4)
- added R16: R, Resistor_SMD:R_0603_1608Metric, F.Cu at (73.6, 64.4)
- added R17: R, Resistor_SMD:R_0603_1608Metric, F.Cu at (75.1, 64.4)
- added R18: R, Resistor_SMD:R_0603_1608Metric, F.Cu at (76.6, 64.4)
- added R20: R, Resistor_SMD:R_0603_1608Metric, F.Cu at (81.5, 58.3)
- added R21: R, Resistor_SMD:R_0603_1608Metric, F.Cu at (81.5, 56.8)
- added R22: R, Resistor_SMD:R_0603_1608Metric, F.Cu at (81.5, 55.3)
- added R23: R, Resistor_SMD:R_0603_1608Metric, F.Cu at (81.5, 53.8)
- added R24: R, Resistor_SMD:R_0603_1608Metric, F.Cu at (81.5, 52.3)
- added R25: R, Resistor_SMD:R_0603_1608Metric, F.Cu at (81.5, 50.8)
- added R26: R, Resistor_SMD:R_0603_1608Metric, F.Cu at (81.5, 49.3)
- added R27: R, Resistor_SMD:R_0603_1608Metric, F.Cu at (81.5, 44.8)
- added R28: R, Resistor_SMD:R_0603_1608Metric, F.Cu at (81.5, 43.3)
- added R3: R, Resistor_SMD:R_0603_1608Metric, F.Cu at (56.4, 54.2)
- added R4: R, Resistor_SMD:R_0603_1608Metric, F.Cu at (56.4, 55.8)
- added R5: R, Resistor_SMD:R_0603_1608Metric, F.Cu at (56.4, 57.4)
- added R6: R, Resistor_SMD:R_0603_1608Metric, F.Cu at (56.4, 58.9)
- added R7: R, Resistor_SMD:R_0603_1608Metric, F.Cu at (81.5, 47.8)
- added R8: R, Resistor_SMD:R_0603_1608Metric, F.Cu at (81.5, 46.3)
- added R9: R, Resistor_SMD:R_0603_1608Metric, F.Cu at (63.1, 64.4)
- R1, R29, R30: footprint Resistor_SMD:R_0805_2012Metric -> Resistor_SMD:R_0603_1608Metric
- R19: value 1k -> R; footprint Resistor_SMD:R_0805_2012Metric -> Resistor_SMD:R_0603_1608Metric
- moved D1 49.4 mm to (97.1, 42.4), turned to 90 degrees
- moved R2 46.7 mm to (94.8, 42.4), turned to 90 degrees
- moved C4 27.6 mm to (49.2, 47.7), turned to -90 degrees
- moved U2 22.6 mm to (52.5, 47.7), turned to 180 degrees
- moved SW1 21.3 mm to (93.0, 64.4)
- moved C3 18.9 mm to (55.8, 47.6), turned to -90 degrees
- moved R1 13.4 mm to (81.5, 61.3), turned to 180 degrees
- moved C2 5.14 mm to (53.8, 40.0), turned to 180 degrees
- moved C1 5.12 mm to (53.3, 42.5), turned to 180 degrees
- moved R30 4.57 mm to (56.4, 62.0), turned to 0 degrees
- moved R29 3.92 mm to (56.4, 60.5), turned to 0 degrees
- moved U1 2.71 mm to (69.5, 49.3)
- moved R19 1.92 mm to (81.5, 59.8), turned to 0 degrees
- moved D2 0.56 mm to (48.8, 65.8)
Connections:
- R1 pad 1: GND -> Net-(R1-Pad1)
- R1 pad 2: Net-(R1-Pad2) -> Net-(U1-IO0)
- R19 pad 1: GND -> /gpio3
- R19 pad 2: Net-(R19-Pad2) -> /GPIO_3
- SW1 pad 1: Net-(R1-Pad2) -> GND
- SW1 pad 2: Net-(U1-IO0) -> Net-(R1-Pad1)
- U1 pad 10: /I2C_SDA -> unconnected-(U1-IO17-Pad10)
- U1 pad 11: /I2C_CLK -> unconnected-(U1-IO18-Pad11)
- U1 pad 15: /SPI_MISO -> unconnected-(U1-IO3-Pad15)
- U1 pad 16: /SPI_CS -> unconnected-(U1-IO46-Pad16)
- U1 pad 17: /SPI_MOSI -> /uart1_rx
- U1 pad 18: /SPI_CLK -> /uart1_tx
- U1 pad 19: /spi3_miso -> /i2c_sda
- U1 pad 20: /IMU_FSYNC -> /i2c_clk
- U1 pad 23: /spi3_mosi -> /spi3_miso
- U1 pad 24: /GPIO_1 -> /spi3_mosi
- U1 pad 25: /GPIO_2 -> /gpio1
- U1 pad 26: Net-(U1-IO45) -> /gpio2
- U1 pad 28: /GPIO_3 -> /gpio3
- U1 pad 29: /GPIO_4 -> /gpio4
- U1 pad 30: /GPIO_5 -> /gpio5
- U1 pad 31: /GPIO_6 -> /gpio6
- U1 pad 32: /GPIO_7 -> /gpio7
- U1 pad 33: /GPIO_8 -> /gpio8
- U1 pad 34: /GPIO_9 -> /gpio9
- U1 pad 35: /GPIO_10 -> /gpio10
- U1 pad 36: /UART1_Rx -> /uart0_rx
- U1 pad 37: /UART1_Tx -> /uart0_tx
- U1 pad 38: /GPIO_11 -> /gpio11
- U1 pad 39: /GPIO_12 -> /gpio12
- U1 pad 4: /ADC_1 -> /adc1_ch3
- U1 pad 5: /ADC_2 -> /adc1_ch4
- U1 pad 6: /ADC_3 -> /adc1_ch5
- U1 pad 7: /ADC_4 -> /adc1_ch6
- U1 pad 8: /UART2_Rx -> unconnected-(U1-IO15-Pad8)
- U1 pad 9: /UART2_Tx -> unconnected-(U1-IO16-Pad9)
- U2 pad 1: /spi3_miso -> /spi2_miso
- U2 pad 12: /spi3_cs -> /spi2_cs
- U2 pad 13: /spi3_clk -> /spi2_clk
- U2 pad 14: /spi3_mosi -> /spi2_mosi
Routing:
- net /GPIO_12: track 0.00 -> 27.4 mm
- net /GPIO_11: track 0.00 -> 26.0 mm, vias 2 -> 3
- net /UART1_Tx: track 0.00 -> 23.9 mm, vias 2 -> 3
- net /UART1_Rx: track 0.00 -> 21.8 mm, vias 2 -> 3
- net /GPIO_10: track 0.00 -> 19.6 mm, vias 2 -> 3
- net /GPIO_9: track 0.00 -> 19.1 mm
- net /GPIO_8: track 0.00 -> 17.8 mm, vias 2 -> 1
- net /SPI_CS: track 0.00 -> 16.9 mm
- net /GPIO_7: track 0.00 -> 15.6 mm
- net /I2C_SDA: track 0.00 -> 15.2 mm
- net /SPI_CLK: track 0.00 -> 13.2 mm
- net /GPIO_6: track 0.00 -> 13.2 mm
- net /UART2_Rx: track 0.00 -> 12.8 mm
- net /I2C_CLK: track 0.00 -> 12.0 mm
- net /GPIO_5: track 0.00 -> 11.3 mm
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