File: hw/kicad/cpu/esp32 s3/esp32 s3.kicad_sch (KiCad schematic)
At the start: 18 parts, among them J1 TOP, J2 BUTTOM, J3 USB_B_Micro, SW1 SW_Push, SW2 SW_Push, U1 ESP32-S3-WROOM-1-N16R2, U2 ICM-42688-P

Commit message: cpu板io电阻
Parts:
- removed SW2: SW_Push, Button_Switch_THT:SW_SPST_Omron_B3F-315x_Angled, symbol Switch:SW_Push
- added R10, R11, R12, R13, R14, R15, R16, R17, R18, R20, R21, R22, R23, R24, R25, R26, R27, R28, R3, R4, R5, R6, R7, R8, R9: R, Resistor_SMD:R_0603_1608Metric, symbol Device:R
- R1, R29, R30: footprint Resistor_SMD:R_0805_2012Metric -> Resistor_SMD:R_0603_1608Metric
- R19: value 1k -> R; footprint Resistor_SMD:R_0805_2012Metric -> Resistor_SMD:R_0603_1608Metric
Connections:
- net ADC_1: now also R3.2; no longer U1.4 (IO4)
- net ADC_2: now also R4.2; no longer U1.5 (IO5)
- net ADC_3: now also R5.2; no longer U1.6 (IO6)
- net ADC_4: now also R6.2; no longer U1.7 (IO7)
- net GND: now also SW1.1; no longer R1.1, R19.1
- net GPIO_1: now also R17.2; no longer U1.24 (IO47)
- net GPIO_10: now also R26.2; no longer U1.35 (IO42)
- net GPIO_11: now also R27.2; no longer U1.38 (IO2)
- net GPIO_12: now also R28.2; no longer U1.39 (IO1)
- net GPIO_2: now also R18.2; no longer U1.25 (IO48)
- net GPIO_3: now also R19.2; no longer U1.28 (IO35)
- net GPIO_4: now also R20.2; no longer U1.29 (IO36)
- net GPIO_5: now also R21.2; no longer U1.30 (IO37)
- net GPIO_6: now also R22.2; no longer U1.31 (IO38)
- net GPIO_7: now also R23.2; no longer U1.32 (IO39)
- net GPIO_8: now also R24.2; no longer U1.33 (IO40)
- net GPIO_9: now also R25.2; no longer U1.34 (IO41)
- net I2C_CLK: now also R12.2; no longer U1.11 (IO18)
- net I2C_SDA: now also R11.2; no longer U1.10 (IO17)
- net IMU_FSYNC: no longer U1.20 (IO12)
- net SPI_CLK: now also R14.2; no longer U1.18 (IO10)
- net SPI_CS: now also R13.2; no longer U1.16 (IO46)
- net SPI_MISO: now also R16.2; no longer U1.15 (IO3)
- net SPI_MOSI: now also R15.2; no longer U1.17 (IO9)
- net UART1_Rx: now also R7.2; no longer U1.36 (RXD0)
- net UART1_Tx: now also R8.2; no longer U1.37 (TXD0)
- net UART2_Rx: now also R9.2; no longer U1.8 (IO15)
- net UART2_Tx: now also R10.2; no longer U1.9 (IO16)
- net spi3_clk: now also R14.1; no longer U2.13 (AP_SCL/AP_SCLK)
- net spi3_cs: now also R13.1; no longer U2.12 (AP_CS)
- net spi3_miso: now also U1.23 (IO21), R16.1; no longer U1.19 (IO11), U2.1 (AP_SDO/AP_AD0)
- net spi3_mosi: now also U1.24 (IO47), R15.1; no longer U1.23 (IO21), U2.14 (AP_SDA/AP_SDIO/AP_SDI)
- net gpio2: now reaches U1.26 (IO45)
- net gpio2: now also R18.1
- net at U1.27 (IO0): now also R1.2; no longer SW1.2
- new net: R1.1, SW1.2
- new net adc1_ch3: R3.1, U1.4 (IO4)
- new net adc1_ch4: R4.1, U1.5 (IO5)
- new net adc1_ch5: R5.1, U1.6 (IO6)
- new net adc1_ch6: R6.1, U1.7 (IO7)
- new net gpio1: R17.1, U1.25 (IO48)
- new net gpio10: R26.1, U1.35 (IO42)
- new net gpio11: R27.1, U1.38 (IO2)
- new net gpio12: R28.1, U1.39 (IO1)
- new net gpio3: R19.1, U1.28 (IO35)
- new net gpio4: R20.1, U1.29 (IO36)
- new net gpio5: R21.1, U1.30 (IO37)
- new net gpio6: R22.1, U1.31 (IO38)
- new net gpio7: R23.1, U1.32 (IO39)
- new net gpio8: R24.1, U1.33 (IO40)
- new net gpio9: R25.1, U1.34 (IO41)
- new net i2c_clk: R12.1, U1.20 (IO12)
- new net i2c_sda: R11.1, U1.19 (IO11)
- new net spi2_clk: U2.13 (AP_SCL/AP_SCLK)
- new net spi2_cs: U2.12 (AP_CS)
- new net spi2_miso: U2.1 (AP_SDO/AP_AD0)
- new net spi2_mosi: U2.14 (AP_SDA/AP_SDIO/AP_SDI)
- new net uart0_rx: R7.1, U1.36 (RXD0)
- new net uart0_tx: R8.1, U1.37 (TXD0)
- new net uart1_rx: R9.1, U1.17 (IO9)
- new net uart1_tx: R10.1, U1.18 (IO10)
Other:
- moved on the sheet: R1, SW1
