File: hw/kicad/app/motor/dc_motor/dc_motor.kicad_pcb (KiCad board)
At the start: 2 copper layers, 40 x 40 mm, 22 parts, among them J1 TOP, J2 Motor 1, J3 Motor 2, J4 Motor 3, J5 BUTTOM, J6 Motor 4, U1 DRV8870DDA, U2 DRV8870DDA, U3 DRV8870DDA, U6 DRV8870DDA

Commit message: Merge from normal
Parts:
- C1, C17, C3, C5: footprint Capacitor_SMD:C_1210_3225Metric -> Capacitor_SMD:CP_Elec_6.3x5.4
- moved C11 7.97 mm to (79.2, 43.5), turned to 90 degrees
- moved C2 7.03 mm to (63.1, 59.2)
- moved C4 6.93 mm to (63.0, 44.7)
- moved C6 6.84 mm to (88.7, 48.4)
- moved C18 6.38 mm to (88.8, 62.9)
- moved C9 6.35 mm to (72.6, 64.1), turned to -90 degrees
- moved C16 5.60 mm to (79.2, 58.1), turned to 90 degrees
- moved C10 4.39 mm to (72.5, 49.7), turned to -90 degrees
- moved U3 3.97 mm to (85.3, 42.8)
- moved C5 3.95 mm to (82.6, 49.6), turned to 180 degrees
- moved J3 3.48 mm to (56.5, 46.7)
- moved J2 3.10 mm to (56.5, 61.2)
- moved U1 3.10 mm to (66.8, 64.8)
- moved C17 2.89 mm to (82.8, 63.9), turned to 180 degrees
- moved J1 2.78 mm to (75.7, 75.2)
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Connections:
- J2 pad 1: /OUT1 -> +3.3V
- J2 pad 2: /OUT2 -> /ENC_1A
- J2 pad 3: GND -> unconnected-(J2-Pin_3-Pad3)
- J2 pad 4: /ENC_1B -> GND
- J2 pad 5: /ENC_1A -> /OUT1
- J2 pad 6: +3.3V -> /OUT2
- J3 pad 1: /OUT3 -> +3.3V
- J3 pad 2: /OUT4 -> /ENC_2A
- J3 pad 3: GND -> unconnected-(J3-Pin_3-Pad3)
- J3 pad 4: /ENC_2B -> GND
- J3 pad 5: /ENC_2A -> /OUT3
- J3 pad 6: +3.3V -> /OUT4
- J4 pad 1: /OUT5 -> +3.3V
- J4 pad 2: /OUT6 -> /ENC_3A
- J4 pad 3: GND -> unconnected-(J4-Pin_3-Pad3)
- J4 pad 4: /ENC_3B -> GND
- J4 pad 5: /ENC_3A -> /OUT5
- J4 pad 6: +3.3V -> /OUT6
- J6 pad 1: /OUT7 -> +3.3V
- J6 pad 2: /OUT8 -> /ENC_4A
- J6 pad 3: GND -> unconnected-(J6-Pin_3-Pad3)
- J6 pad 4: /ENC_4B -> GND
- J6 pad 5: /ENC_4A -> /OUT7
- J6 pad 6: +3.3V -> /OUT8
Routing:
- net +BATT: track 44.8 -> 119.5 mm, vias 10 -> 12
- net +3.3V: track 103.0 -> 166.8 mm, vias 11 -> 7
- net /GPIO_5: track 5.13 -> 39.8 mm
- net /GPIO_6: track 4.45 -> 37.5 mm
- net /GPIO_3: track 2.84 -> 31.8 mm
- net /ENC_4A: track 10.3 -> 36.3 mm
- net /ENC_1A: track 7.14 -> 33.0 mm
- net /ENC_2A: track 19.5 -> 44.1 mm
- net /ENC_3A: track 23.3 -> 45.6 mm
- net /GPIO_4: track 3.55 -> 25.1 mm
- net /GPIO_7: track 4.27 -> 24.2 mm
- net /GPIO_8: track 3.56 -> 22.2 mm
- net /GPIO_1: track 5.90 -> 17.2 mm
- net /GPIO_2: track 2.66 -> 9.98 mm
- net /OUT2: track 10.2 -> 6.52 mm
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Other:
- board size 40 x 40 mm -> 45 x 45 mm
- board text added: "Pindar v1.2 (App) DC Motor v1.2"
- board text removed: "Pindar v1.0 Type APP Mecanum wheel v1.0"
