File: hw/kicad/base/power_16V/power_16V.kicad_sch (KiCad schematic)
At the start: 34 parts, among them J1 USB_B_Micro, J2 XT30PW-M, J3 TOP, J4 BUTTOM, U1 LM2596S-5, U2 LM1117MP-3.3, U3 CP2104

Commit message: 尽力改成40mmx40mm
Parts:
- removed C10: 220uF, Capacitor_SMD:CP_Elec_6.3x7.7, symbol Device:C_Polarized
- C1: value 220uF -> 100uF
Connections:
- net UART3_Rx is gone; now on net I2C_SDA: J3.9 (Pin_9), J4.10 (Pin_10)
- net UART3_Tx is gone; now on net I2C_CLK: J3.10 (Pin_10), J4.9 (Pin_9)
- net +3.3V: now also R3.1; no longer D7.2 (A)
- net GND: now also D7.2 (A); no longer R3.1
- net GPIO_1: now also J3.15 (Pin_15), J4.16 (Pin_16); no longer J3.17 (Pin_17), J4.18 (Pin_18)
- net GPIO_10: now also J3.24 (Pin_24), J4.23 (Pin_23); no longer J3.26 (Pin_26), J4.25 (Pin_25)
- net GPIO_2: now also J3.16 (Pin_16), J4.15 (Pin_15); no longer J3.18 (Pin_18), J4.17 (Pin_17)
- net GPIO_3: now also J3.17 (Pin_17), J4.18 (Pin_18); no longer J3.19 (Pin_19), J4.20 (Pin_20)
- net GPIO_4: now also J3.18 (Pin_18), J4.17 (Pin_17); no longer J3.20 (Pin_20), J4.19 (Pin_19)
- net GPIO_5: now also J3.19 (Pin_19), J4.20 (Pin_20); no longer J3.21 (Pin_21), J4.22 (Pin_22)
- net GPIO_6: now also J3.20 (Pin_20), J4.19 (Pin_19); no longer J3.22 (Pin_22), J4.21 (Pin_21)
- net GPIO_7: now also J3.21 (Pin_21), J4.22 (Pin_22); no longer J3.23 (Pin_23), J4.24 (Pin_24)
- net GPIO_8: now also J3.22 (Pin_22), J4.21 (Pin_21); no longer J3.24 (Pin_24), J4.23 (Pin_23)
- net GPIO_9: now also J3.23 (Pin_23), J4.24 (Pin_24); no longer J3.25 (Pin_25), J4.26 (Pin_26)
- net I2C_CLK: no longer J3.12 (Pin_12), J4.11 (Pin_11)
- net I2C_SDA: no longer J3.11 (Pin_11), J4.12 (Pin_12)
- net SPI_CLK: now also J3.12 (Pin_12), J4.11 (Pin_11); no longer J3.14 (Pin_14), J4.13 (Pin_13)
- net SPI_CS: now also J3.11 (Pin_11), J4.12 (Pin_12); no longer J3.13 (Pin_13), J4.14 (Pin_14)
- net SPI_MISO: now also J3.14 (Pin_14), J4.13 (Pin_13); no longer J3.16 (Pin_16), J4.15 (Pin_15)
- net SPI_MOSI: now also J3.13 (Pin_13), J4.14 (Pin_14); no longer J3.15 (Pin_15), J4.16 (Pin_16)
- new net GPIO_11: J3.25 (Pin_25), J4.26 (Pin_26)
- new net GPIO_12: J3.26 (Pin_26), J4.25 (Pin_25)
Other:
- moved on the sheet: D7, R3

Commit message: Merge from normal
Parts:
- added C10: 220uF, Capacitor_SMD:CP_Elec_6.3x7.7, symbol Device:C_Polarized
- added C11, C12: 0.1uF, Capacitor_SMD:C_0805_2012Metric, symbol Device:C
- added U4: ACS712xLCTR-05B, Package_SO:SOIC-8_3.9x4.9mm_P1.27mm, symbol Sensor_Current:ACS712xLCTR-05B
- C1: value 100uF -> 220uF
- R1, R2: footprint Resistor_SMD:R_0805_2012Metric -> Resistor_SMD:R_0603_1608Metric
- R4, R5: value 22 -> 100
Connections:
- net GPIO_11 is gone; now on net GPIO_9: J3.25 (Pin_25), J4.26 (Pin_26)
- net GPIO_12 is gone; now on net GPIO_10: J3.26 (Pin_26), J4.25 (Pin_25)
- net +3.3V: now also D7.2 (A); no longer R3.1
- net +BATT: now also C10.1, U4.3 (IP-), U4.4 (IP-); no longer J2.2 (-)
- net ADC_2: now also C12.1, U4.7 (VIOUT)
- net GND: now also J2.2 (-), R3.1, C10.2, C11.2, C12.2, U4.5 (GND); no longer D7.2 (A), J2.1 (+)
- net GPIO_1: now also J3.17 (Pin_17), J4.18 (Pin_18); no longer J3.15 (Pin_15), J4.16 (Pin_16)
- net GPIO_10: no longer J3.24 (Pin_24), J4.23 (Pin_23)
- net GPIO_2: now also J3.18 (Pin_18), J4.17 (Pin_17); no longer J3.16 (Pin_16), J4.15 (Pin_15)
- net GPIO_3: now also J3.19 (Pin_19), J4.20 (Pin_20); no longer J3.17 (Pin_17), J4.18 (Pin_18)
- net GPIO_4: now also J3.20 (Pin_20), J4.19 (Pin_19); no longer J3.18 (Pin_18), J4.17 (Pin_17)
- net GPIO_5: now also J3.21 (Pin_21), J4.22 (Pin_22); no longer J3.19 (Pin_19), J4.20 (Pin_20)
- net GPIO_6: now also J3.22 (Pin_22), J4.21 (Pin_21); no longer J3.20 (Pin_20), J4.19 (Pin_19)
- net GPIO_7: now also J3.23 (Pin_23), J4.24 (Pin_24); no longer J3.21 (Pin_21), J4.22 (Pin_22)
- net GPIO_8: now also J3.24 (Pin_24), J4.23 (Pin_23); no longer J3.22 (Pin_22), J4.21 (Pin_21)
- net GPIO_9: no longer J3.23 (Pin_23), J4.24 (Pin_24)
- net I2C_CLK: now also J3.12 (Pin_12), J4.11 (Pin_11); no longer J3.10 (Pin_10), J4.9 (Pin_9)
- net I2C_SDA: now also J3.11 (Pin_11), J4.12 (Pin_12); no longer J3.9 (Pin_9), J4.10 (Pin_10)
- net SPI_CLK: now also J3.14 (Pin_14), J4.13 (Pin_13); no longer J3.12 (Pin_12), J4.11 (Pin_11)
- net SPI_CS: now also J3.13 (Pin_13), J4.14 (Pin_14); no longer J3.11 (Pin_11), J4.12 (Pin_12)
- net SPI_MISO: now also J3.16 (Pin_16), J4.15 (Pin_15); no longer J3.14 (Pin_14), J4.13 (Pin_13)
- net SPI_MOSI: now also J3.15 (Pin_15), J4.16 (Pin_16); no longer J3.13 (Pin_13), J4.14 (Pin_14)
- net DCDC_+5V: now reaches C7.1, C8.1, D6.2 (A), L1.2, U1.4 (FB)
- net DCDC_+5V: now also U4.8 (VCC)
- new net: C11.1, U4.6 (FILTER)
- new net +BATT_IN: J2.1 (+), U4.1 (IP+), U4.2 (IP+)
- new net UART3_Rx: J3.9 (Pin_9), J4.10 (Pin_10)
- new net UART3_Tx: J3.10 (Pin_10), J4.9 (Pin_9)
Other:
- moved on the sheet: C1, C2, C3, C6, C7, C8, D3, D6, D7, J2, L1, R3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
